Commit message: add goal marker

File: urdf/franka_paddle.urdf (robot description, URDF)
Before this commit: robot panda, 10 links, 9 joints
Joints:
- joint panda_paddle_joint: origin xyz=-0.14 0 -0.02 rpy=0 0 0 -> xyz=0.0 0.1 0.0 rpy=0 0 0

Commit message: add prismatics at 0

File: urdf/franka_paddle.urdf (robot description, URDF)
Before this commit: robot panda, 10 links, 9 joints
Links:
- added link sliderx_link; visual box size=0.001 0.001 0.001
- added link slidery_link; visual box size=0.001 0.001 0.001
Joints:
- added joint panda_sliderx: type prismatic, parent panda_paddle, child sliderx_link, origin xyz=0 0 0 rpy=0 0 0, axis 1 0 0, limit lower=-0.075 upper=0.075 effort=100 velocity=0.5
- added joint panda_slidery: type prismatic, parent sliderx_link, child slidery_link, origin xyz=0 0 0 rpy=0 0 0, axis 0 1 0, limit lower=-0.1 upper=0.1 effort=100 velocity=0.5
